Commit message: Made the visual and collision geometries uniform

File: gym_env/assets/cylinder.urdf (robot description, URDF)
Before this commit: robot cylinder.urdf, 1 links, 0 joints
Links:
- link cylinder: geometry collision cylinder length=2.0 radius=0.2; visual cylinder length=2.0 radius=0.2

Commit message: Added Walls and Tress in sim

File: gym_env/assets/cylinder.urdf (robot description, URDF)
Before this commit: robot cylinder.urdf, 1 links, 0 joints
Links:
- link cylinder: geometry collision cylinder length=2.0 radius=0.3; visual mesh filename=bark.obj scale=.5 .5 .5
